File: Hardware/SmartMeter.brd (EAGLE design)
At the start: 31.7 x 58.2 mm, 25 parts, among them J1 J0011D01

Commit message: Cleanup
Parts:
- C1, C2: value (none) -> 100nF
- IC1: value (none) -> LM1117
- Q1, Q2: value (none) -> SI2302
- R1, R2, R3, R4, R5, R6, R7: value (none) -> 12K
- R8, R9: value (none) -> 470R
Changed lines of the file:
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@@
 </autorouter>
 <elements>
-<element name="C1" library="rc-master-smd" package="C0805MP" value="" x="6.985" y="52.705">
+<element name="C1" library="rc-master-smd" package="C0805MP" value="100nF" x="6.985" y="52.705">
 <attribute name="NAME" x="5.3975" y="53.6575" size="0.8128" layer="25" ratio="18"/>
 <attribute name="VALUE" x="5.3975" y="51.435" size="0.4064" layer="27" ratio="10"/>
 </element>
-<element name="C2" library="rc-master-smd" package="C0805MP" value="" x="7.62" y="42.164" rot="R180">
+<element name="C2" library="rc-master-smd" package="C0805MP" value="100nF" x="7.62" y="42.164" rot="R180">
 <attribute name="NAME" x="9.2075" y="41.2115" size="0.8128" layer="25" ratio="18" rot="R180"/>
 <attribute name="VALUE" x="9.2075" y="43.434" size="0.4064" layer="27" ratio="10" rot="R180"/>
@@
 <attribute name="NAME" x="10.672" y="9.112" size="1.27" layer="25"/>
 </element>
-<element name="Q1" library="epic" package="SOT-23" value="" x="5.969" y="33.655" rot="R90">
+<element name="Q1" library="epic" package="SOT-23" value="SI2302" x="5.969" y="33.655" rot="R90">
 <attribute name="NAME" x="2.667" y="32.258" size="1.27" layer="25" ratio="10" rot="R90"/>
 <attribute name="VALUE" x="4.191" y="32.258" size="1.27" layer="27" ratio="10" rot="R90"/>
 </element>
-<element name="R1" library="passives" package="0805_RES" value="" x="22.733" y="51.308" rot="R180">
+<element name="R1" library="passives" package="0805_RES" value="12K" x="22.733" y="51.308" rot="R180">
 <attribute name="NAME" x="22.733" y="51.578" size="1.016" layer="25" font="vector" ratio="12" rot="R180" align="bottom-center"/>
 <attribute name="VALUE" x="22.733" y="53.308" size="1.016" layer="27" font="vector" ratio="12" rot="R180" align="bottom-center"/>
 </element>
-<element name="R2" library="passives" package="0805_RES" value="" x="7.366" y="38.608" rot="R180">
+<element name="R2" library="passives" package="0805_RES" value="12K" x="7.366" y="38.608" rot="R180">
 <attribute name="NAME" x="7.366" y="37.608" size="1.016" layer="25" font="vector" ratio="12" rot="R180" align="bottom-center"/>
 <attribute name="VALUE" x="7.366" y="40.608" size="1.016" layer="27" font="vector" ratio="12" rot="R180" align="bottom-center"/>
 </element>
-<element name="R3" library="passives" package="0805_RES" value="" x="13.208" y="13.843">
+<element name="R3" library="passives" package="0805_RES" value="12K" x="13.208" y="13.843">
 <attribute name="NAME" x="13.208" y="14.843" size="1.016" layer="25" font="vector" ratio="12" align="bottom-center"/>
 <attribute name="VALUE" x="13.208" y="11.843" size="1.016" layer="27" font="vector" ratio="12" align="bottom-center"/>
 </element>
-<element name="R4" library="passives" package="0805_RES" value="" x="17.399" y="13.843">
+<element name="R4" library="passives" package="0805_RES" value="12K" x="17.399" y="13.843">
 <attribute name="NAME" x="17.399" y="14.843" size="1.016" layer="25" font="vector" ratio="12" align="bottom-center"/>
 <attribute name="VALUE" x="17.399" y="11.843" size="1.016" layer="27" font="vector" ratio="12" align="bottom-center"/>
 </element>
-<element name="R5" library="passives" package="0805_RES" value="" x="29.972" y="5.588" rot="R270">
+<element name="R5" library="passives" package="0805_RES" value="12K" x="29.972" y="5.588" rot="R270">
 <attribute name="NAME" x="30.972" y="5.588" size="1.016" layer="25" font="vector" ratio="12" rot="R270" align="bottom-center"/>
 <attribute name="VALUE" x="27.972" y="5.588" size="1.016" layer="27" font="vector" ratio="12" rot="R270" align="bottom-center"/>
 </element>
-<element name="R6" library="passives" package="0805_RES" value="" x="30.988" y="22.479" rot="R90">
+<element name="R6" library="passives" package="0805_RES" value="12K" x="30.988" y="22.479" rot="R90">
 <attribute name="NAME" x="29.988" y="22.479" size="1.016" layer="25" font="vector" ratio="12" rot="R90" align="bottom-center"/>
 <attribute name="VALUE" x="32.988" y="22.479" size="1.016" layer="27" font="vector" ratio="12" rot="R90" align="bottom-center"/>
 </element>
-<element name="R7" library="passives" package="0805_RES" value="" x="29.972" y="11.938" rot="R90">
+<element name="R7" library="passives" package="0805_RES" value="12K" x="29.972" y="11.938" rot="R90">
 <attribute name="NAME" x="28.972" y="11.938" size="1.016" layer="25" font="vector" ratio="12" rot="R90" align="bottom-center"/>
 <attribute name="VALUE" x="31.972" y="11.938" size="1.016" layer="27" font="vector" ratio="12" rot="R90" align="bottom-center"/>
 </element>
-<element name="R8" library="passives" package="0805_RES" value="" x="9.144" y="28.702" rot="R270">
+<element name="R8" library="passives" package="0805_RES" value="470R" x="9.144" y="28.702" rot="R270">
 <attribute name="NAME" x="10.144" y="28.702" size="1.016" layer="25" font="vector" ratio="12" rot="R270" align="bottom-center"/>
 <attribute name="VALUE" x="7.144" y="28.702" size="1.016" layer="27" font="vector" ratio="12" rot="R270" align="bottom-center"/>
 </element>
-<element name="R9" library="passives" package="0805_RES" value="" x="9.144" y="16.002" rot="R90">
+<element name="R9" library="passives" package="0805_RES" value="470R" x="9.144" y="16.002" rot="R90">
 <attribute name="NAME" x="8.144" y="16.002" size="1.016" layer="25" font="vector" ratio="12" rot="R90" align="bottom-center"/>
 <attribute name="VALUE" x="11.144" y="16.002" size="1.016" layer="27" font="vector" ratio="12" rot="R90" align="bottom-center"/>
@@
 <attribute name="VALUE" x="13.128" y="13.754" size="1.4224" layer="27"/>
 </element>
-<element name="IC1" library="v-reg-3" package="SOT223" value="" x="9.017" y="46.736" rot="R90">
+<element name="IC1" library="v-reg-3" package="SOT223" value="LM1117" x="9.017" y="46.736" rot="R90">
 <attribute name="NAME" x="8.9662" y="44.196" size="1.27" layer="25" rot="R90"/>
 <attribute name="VALUE" x="10.3378" y="44.196" size="1.27" layer="27" rot="R90"/>
@@
 <attribute name="NAME" x="11.4935" y="40.005" size="0.8128" layer="25" ratio="18" rot="R90"/>
 </element>
-<element name="Q2" library="epic" package="SOT-23" value="" x="17.018" y="40.386" rot="R180">
+<element name="Q2" library="epic" package="SOT-23" value="SI2302" x="17.018" y="40.386" rot="R180">
 <attribute name="NAME" x="18.415" y="37.084" size="1.27" layer="25" ratio="10" rot="R180"/>
 <attribute name="VALUE" x="18.415" y="38.608" size="1.27" layer="27" ratio="10" rot="R180"/>
